Commit message: Change core URDF

File: description/robot_core.xacro (robot description, xacro)
@@ -45,4 +45,7 @@
         </xacro:inertial_box>
     </link>
+    <gazebo reference="chassis_link">
+        <material>Gazebo/White</material>
+    </gazebo>
     <!--Left Wheel Joint-->
     <joint name="left_wheel_joint" type="continuous">
@@ -69,4 +72,7 @@
         </xacro:inertial_cylinder>
     </link>
+    <gazebo reference="left_wheel_link">
+        <material>Gazebo/Blue</material>
+    </gazebo>
     <!--Right Wheel Joint-->
     <joint name="right_wheel_joint" type="continuous">
@@ -93,4 +99,7 @@
         </xacro:inertial_cylinder>
     </link>
+    <gazebo reference="right_wheel_link">
+        <material>Gazebo/Blue</material>
+    </gazebo>
     <!--Caster Wheel Joint-->
     <joint name="caster_wheel_joint" type="fixed">
@@ -116,3 +125,8 @@
         </xacro:inertial_sphere>
     </link>
+    <gazebo reference="caster_wheel_link">
+        <material>Gazebo/Black</material>
+        <mu1 value="0.001" />
+        <mu2 value="0.001" />
+    </gazebo>
 </robot>

Commit message: Add lidar description

File: description/robot_core.xacro (robot description, xacro)
@@ -17,4 +17,8 @@
     <material name="black">
         <color rgba="0 0 0 1" />
+    </material>
+    <!--Red Color-->
+    <material name="red">
+        <color rgba="1 0 0 1" />
     </material>
     <!--Base Link-->
