Commit message: Add camera description

File: description/lidar.xacro (robot description, xacro)
@@ -26,5 +26,5 @@
         <sensor name="laser" type="ray">
             <pose> 0 0 0 0 0 0 </pose>
-            <visualize>true</visualize>
+            <visualize>false</visualize>
             <update_rate>10</update_rate>
             <ray>

File: description/robot_core.xacro (robot description, xacro)
@@ -5,8 +5,4 @@
     <material name="white">
         <color rgba="1 1 1 1" />
-    </material>
-    <!--Orange Color-->
-    <material name="orange">
-        <color rgba="1 0.3 0.1 1" />
     </material>
     <!--Blue Color-->
